Commit message: Completely refactor servo def

File: src/herkulex/herkulex_description/urdf/drs_x01.xacro (robot description, xacro)
@@ -1,58 +1,172 @@
 <?xml version="1.0" encoding="UTF-8"?>
-<robot xmlns:controller="http://playerstage.sourceforge.net/gazebo/xmlschema/#controller"
-	xmlns:interface="http://playerstage.sourceforge.net/gazebo/xmlschema/#interface"
-	xmlns:sensor="http://playerstage.sourceforge.net/gazebo/xmlschema/#sensor"
-	xmlns:xacro="http://ros.org/wiki/xacro">
-	<xacro:macro name="x01"
-		params="name parent minPosition maxPosition maxVelocity *origin">
+<robot xmlns:controller="http://playerstage.sourceforge.net/gazebo/xmlschema/#controller" xmlns:interface="http://playerstage.sourceforge.net/gazebo/xmlschema/#interface"
+	xmlns:sensor="http://playerstage.sourceforge.net/gazebo/xmlschema/#sensor" xmlns:xacro="http://ros.org/wiki/xacro">
+	<xacro:macro name="drs_x01" params="name parent mountTop mountBottom mountBack mountAxel minPosition maxPosition maxVelocity *origin">
+		<xacro:mount name="${name}_mount" parent="${parent}">
+			<insert_block name="origin" />
+		</xacro:mount>
+		<xacro:__drs_x01_box skipBottom="${mountBottom}" skipTop="${mountTop}" skipAxel="${mountAxel}" skipBack="${mountBack}"
+			name="${name}" />
+		<joint name="${name}_box_joint" type="fixed">
+			<xacro:if value="${mountBack}">
+				<origin xyz="0 0 0.019" rpy="1.57079 0 -1.57079" />
+			</xacro:if>
+			<xacro:if value="${mountBottom}">
+				<origin xyz="0.025 0 0" rpy="0 1.57079 0" />
+			</xacro:if>
+			<xacro:if value="${mountTop}">
+				<origin xyz="-0.025 0 0" rpy="0 -1.57079 0" />
+			</xacro:if>
+			<xacro:if value="${mountAxel}">
+				<origin xyz="-0.012 0 0.019" rpy="1.57079 0 0" />
+			</xacro:if>
+			<xacro:if value="${mountAxel}">
+				<parent link="${name}_box_axel_link" />
+			</xacro:if>
+			<xacro:unless value="${mountAxel}">
+				<parent link="${name}_mount_link" />
+			</xacro:unless>
+			<child link="${name}_box_link" />
+		</joint>
+		<xacro:__drs_x01_axel name="${name}" mountAxel="${mountAxel}" />
+		<joint name="${name}_axel_box_joint" type="revolute">
+			<xacro:if value="${mountAxel}">
+				<parent link="${name}_axel_box_link" />
+				<child link="${name}_box_axel_link" />
+				<origin xyz="0 0 0" rpy="0 0 0" />
+			</xacro:if>
+			<xacro:unless value="${mountAxel}">
+				<parent link="${name}_box_axel_link" />
+				<child link="${name}_axel_box_link" />
+				<origin xyz="0 0 0" rpy="0 0 0" />
+			</xacro:unless>
+			<axis xyz="0 0 1" />
+			<limit effort="0" lower="-1.5707" upper="1.5707" velocity="1" />
+		</joint>
+		<!-- Gazebo Config -->
+		<transmission name="${name}_trans">
+			<type>transmission_interface/SimpleTransmission</type>
+			<joint name="${name}_joint">
+				<hardwareInterface>PositionJointInterface</hardwareInterface>
+			</joint>
+			<actuator name="${name}_motor">
+				<hardwareInterface>PositionJointInterface</hardwareInterface>
+				<mechanicalReduction>1</mechanicalReduction>
+			</actuator>
+		</transmission>
+		<gazebo reference="${name}_box_link">
+			<material>Gazebo/White</material>
+		</gazebo>
+		<gazebo reference="${name}_box_axel_link">
+			<material>Gazebo/White</material>
+		</gazebo>
+	</xacro:macro>
+	<xacro:macro name="__drs_x01_box" params="name skipBack skipBottom skipTop skipAxel">
 		<link name="${name}_box_link">
 			<visual>
-				<geometry name="x01mesh">
-					<mesh filename="package://herkulex_description/meshes/x01_box_plain.stl"
-						scale="0.001 0.001 0.001" />
+				<geometry name="x01">
+					<box size="0.050 0.038 0.032" />
 				</geometry>
-				<material name="plastic_black">
-					<color rgba="0.33 0.33 0.33 1" />
-				</material>
-				<origin rpy="-1.57075 1.57075 0" xyz="0 0 0.025" />
+				<material name="plastic_black" />
 			</visual>
 			<inertial>
 				<mass value="0.01" />
-				<inertia ixx="0.001" ixy="0.0" ixz="0.0" iyy="0.001" iyz="0.0"
-					izz="0.001" />
+				<inertia ixx="0.001" ixy="0.0" ixz="0.0" iyy="0.001" iyz="0.0" izz="0.001" />
 			</inertial>
 			<collision>
-				<geometry name="x01simple">
+				<geometry name="x01">
 					<box size="0.050 0.038 0.032" />
 				</geometry>
 			</collision>
 		</link>
-		<link name="${name}_link">
+		<xacro:unless value="${skipBack}">
+			<xacro:mount name="${name}_box_back" parent="${name}_box">
+				<origin xyz="0 0.019 0" rpy="1.57079 0 0" />
+			</xacro:mount>
+		</xacro:unless>
+		<xacro:unless value="${skipBottom}">
+			<xacro:mount name="${name}_box_bottom" parent="${name}_box">
+				<origin xyz="0.025 0 0" rpy="0 1.57079 0" />
+			</xacro:mount>
+		</xacro:unless>
+		<xacro:unless value="${skipTop}">
+			<xacro:mount name="${name}_box_top" parent="${name}_box">
+				<origin xyz="-0.025 0 0" rpy="0 -1.57079 0" />
+			</xacro:mount>
+		</xacro:unless>
+		<xacro:unless value="${skipAxel}">
+			<xacro:mount name="${name}_box_axel" parent="${name}_box">
+				<origin xyz="-0.012 0.019 0" rpy="1.57075 0 3.14159" />
+			</xacro:mount>
+		</xacro:unless>
+		<xacro:if value="${skipAxel}">
+			<link name="${name}_box_axel_link">
+			<visual>
+				<origin xyz="0 0 0" rpy="0 0 0" />
+				<geometry>
+					<cylinder length="0.001" radius="0.01" />
+				</geometry>
+				<material name="orange" />
+			</visual></link>
+		</xacro:if>
+	</xacro:macro>
+	<xacro:macro name="__drs_x01_axel" params="name mountAxel">
+		<link name="${name}_axel_box_link">
 			<visual>
 				<geometry>
 					<cylinder length="0.005" radius="0.011" />
 				</geometry>
-				<material name="plastic_white">
-					<color rgba="0.9 0.9 0.9 1" />
-				</material>
-				<origin rpy="0 1.57075 0" xyz="0.0025 0 0" />
+				<material name="plastic_white" />
 			</visual>
 			<inertial>
 				<mass value="0.001" />
-				<inertia ixx="0.001" ixy="0.0" ixz="0.0" iyy="0.001" iyz="0.0"
-					izz="0.001" />
+				<inertia ixx="0.001" ixy="0.0" ixz="0.0" iyy="0.001" iyz="0.0" izz="0.001" />
 			</inertial>
+			<collision>
+				<geometry>
+					<cylinder length="0.005" radius="0.011" />
+				</geometry>
+			</collision>
 		</link>
-		<joint name="${name}_joint" type="revolute">
-			<parent link="${name}_box_link" />
-			<child link="${name}_link" />
-			<origin xyz="0.0165 0 0.037" />
-			<axis xyz="1 0 0" />
+		<xacro:if value="${mountAxel}">
+			<xacro:mount name="${name}_axel" parent="${name}_mount">
+				<origin xyz="0 0 -0.0025" rpy="0 0 0" />
+			</xacro:mount>
+			<joint name="${name}_axel0_joint" type="fixed">
+				<parent link="${name}_axel_link" />
+				<child link="${name}_axel_box_link" />
+				<origin xyz="0 0 0" rpy="0 0 1.57079" />
+			</joint>
+		</xacro:if>
+		<xacro:unless value="${mountAxel}">
+			<xacro:mount name="${name}_axel" parent="${name}_axel_box">
+				<origin xyz="0 0 0.0025" rpy="0 0 1.57079" />
+			</xacro:mount>
+		</xacro:unless>
+	</xacro:macro>
+	<xacro:macro name="drs_x01_axel" params="name parent minPosition maxPosition maxVelocity *origin">
+		<xacro:mount name="${name}_mount" parent="${parent}">
+			<insert_block name="origin" />
+		</xacro:mount>
+		<xacro:__drs_x01_box skip="" name="${name}" />
+		<xacro:__drs_x01_axel name="${name}" />
+		<joint name="${name}_axel_joint" type="fixed">
+			<origin rpy="0 0 0" xyz="0 0 0" />
+			<parent link="${name}_mount_link" />
+			<child link="${name}_axel_link" />
+		</joint>
+		<joint name="${name}_joint" type="fixed">
+			<parent link="${name}_axel_link" />
+			<child link="${name}_box_axel0_link" />
+			<origin xyz="0 0 -0.001" rpy="0 0 0" />
+			<axis xyz="0 0 1" />
 			<limit effort="0" lower="-1.5707" upper="1.5707" velocity="1" />
 		</joint>
-		<joint name="${name}_box_joint" type="fixed">
-			<parent link="${parent}_link" />
+		<link name="${name}_box_axel_link">
+		</link>
+		<joint name="${name}_axel_joint" type="fixed">
+			<parent link="${name}_box_axel_link" />
 			<child link="${name}_box_link" />
-			<insert_block name="origin" />
+			<origin xyz="-0.012 0 0.025" rpy="1.57075 0 3.14159" />
 		</joint>
 		<!-- Gazebo Config -->
@@ -70,86 +184,5 @@
 			<material>Gazebo/FlatBlack</material>
 		</gazebo>
-		<gazebo reference="${name}_link">
-			<material>Gazebo/White</material>
-		</gazebo>
-	</xacro:macro>
-	<xacro:macro name="x01inverted"
-		params="name parent minPosition maxPosition maxVelocity *origin">
-		<link name="${name}_box_link">
-			<visual>
-				<geometry name="x01mesh">
-					<mesh filename="package://dynamixel_description/meshes/x01_box_plain.stl"
-						scale="0.001 0.001 0.001" />
-				</geometry>
-				<material name="plastic_black" />
-				<origin rpy="1.57075 0 3.14159" xyz="-0.012 0 0.019" />
-			</visual>
-			<inertial>
-				<mass value="0.01" />
-				<origin rpy="0 0 0" xyz="-0.012 0 0.019" />
-				<inertia ixx="0.001" ixy="0.0" ixz="0.0" iyy="0.001" iyz="0.0"
-					izz="0.001" />
-			</inertial>
-			<collision>
-				<origin rpy="1.57075 0 3.14159" xyz="-0.012 0 0.019" />
-				<geometry name="x01simple">
-					<box size="0.050 0.038 0.032" />
-				</geometry>
-			</collision>
-		</link>
-		<link name="${name}_cyl_link">
-			<visual>
-				<geometry>
-					<cylinder length="0.005" radius="0.011" />
-				</geometry>
-				<material name="plastic_white" />
-				<origin rpy="0 0 0" xyz="0 0 0.0025" />
-			</visual>
-			<inertial>
-				<mass value="0.001" />
-				<inertia ixx="0.001" ixy="0.0" ixz="0.0" iyy="0.001" iyz="0.0"
-					izz="0.001" />
-				<origin rpy="0 0 0" xyz="0 0 0.0025" />
-			</inertial>
-			<collision>
-				<geometry>
-					<cylinder length="0.005" radius="0.011" />
-					<origin rpy="0 0 0" xyz="0 0 0.0025" />
-				</geometry>
-			</collision>
-		</link>
-		<link name="${name}_link"></link>
-		<joint name="${name}_joint" type="revolute">
-			<parent link="${name}_cyl_link" />
-			<child link="${name}_box_link" />
-			<origin xyz="0 0 0" />
-			<axis xyz="0 0 1" />
-			<limit effort="0" lower="-1.5707" upper="1.5707" velocity="1" />
-		</joint>
-		<joint name="${name}_cyl_joint" type="fixed">
-			<parent link="${parent}_link" />
-			<child link="${name}_cyl_link" />
-			<insert_block name="origin" />
-		</joint>
-		<joint name="${name}_box_joint" type="fixed">
-			<parent link="${name}_box_link" />
-			<child link="${name}_link" />
-			<origin xyz="0 0 0.038" />
-		</joint>
-		<!-- Gazebo Config -->
-		<transmission name="${name}_trans">
-			<type>transmission_interface/SimpleTransmission</type>
-			<joint name="${name}_joint">
-				<hardwareInterface>PositionJointInterface</hardwareInterface>
-			</joint>
-			<actuator name="${name}_motor">
-				<hardwareInterface>PositionJointInterface</hardwareInterface>
-				<mechanicalReduction>1</mechanicalReduction>
-			</actuator>
-		</transmission>
-		<gazebo reference="${name}_box_link">
-			<material>Gazebo/FlatBlack</material>
-		</gazebo>
-		<gazebo reference="${name}_cyl_link">
+		<gazebo reference="${name}_box_axel_link">
 			<material>Gazebo/White</material>
 		</gazebo>

File: src/kaspar_description/urdf/kaspar.xacro (robot description, xacro)
@@ -5,6 +5,6 @@
 	<xacro:property name="mass" value="10" />
 	<!-- Import joint description -->
-	<xacro:include filename="$(find dynamixel_description)/urdf/dynamixel_ax12.xacro" />
-	<xacro:include filename="$(find dynamixel_description)/urdf/fp04_02.xacro" />
+	<xacro:include filename="$(find herkulex_description)/urdf/drs_x01.xacro" />
+	<xacro:include filename="$(find herkulex_description)/urdf/mount.xacro" />
 	<!-- Import individual part macros -->
 	<xacro:include filename="$(find kaspar_description)/urdf/kaspar_arm.xacro" />
@@ -22,16 +22,34 @@
 		<origin rpy="0 0 0" xyz="0 0 0" />
 	</xacro:leg_v0>
+	<xacro:foot_v0 name="foot_l" parent="leg_l_foot">
+		<origin rpy="0 0 0" xyz="0 0 0" />
+	</xacro:foot_v0>
 	<xacro:leg_v0 name="leg_r" parent="base_leg_r">
 		<origin rpy="0 0 0" xyz="0 0 0" />
 	</xacro:leg_v0>
-	<joint name="base_torso_joint" type="revolute">
-		<parent link="base_top_link" />
-		<child link="base_torso_joint_link" />
-		<axis xyz="0 0 1" />
-		<limit effort="0" lower="-1.5707" upper="1.5707" velocity="1" />
-	</joint>
-	<link name="base_torso_joint_link" />
-	<xacro:torso_v0 name="torso" parent="base_torso_joint">
+	<xacro:foot_v0 name="foot_r" parent="leg_r_foot">
+		<origin rpy="0 0 0" xyz="0 0 0" />
+	</xacro:foot_v0>
+	<xacro:torso_v0 name="torso" parent="base_top">
 		<origin rpy="0 0 0" xyz="0 0 0" />
 	</xacro:torso_v0>
+	<xacro:arm_v0 name="arm_r" parent="torso_arm_r">
+		<origin rpy="0 0 0" xyz="0 0 0" />
+	</xacro:arm_v0>
+	<!--
+	<xacro:hand_v0 name="hand_r" parent="torso_arm_r_hand">
+		<origin rpy="0 0 0" xyz="0 0 0" />
+	</xacro:hand_v0>
+	<xacro:arm_v0 name="arm_l" parent="torso_arm_l">
+		<origin rpy="0 0 0" xyz="0 0 0" />
+	</xacro:arm_v0>
+	<xacro:hand_v0 name="hand_l" parent="torso_arm_l_hand">
+		<origin rpy="0 0 0" xyz="0 0 0" />
+	</xacro:hand_v0>
+	<xacro:neck_v0 name="neck" parent="torso_top">
+		<origin rpy="0 0 0" xyz="0 0 0" />
+	</xacro:neck_v0>
+	<xacro:head_v0 name="head" parent="neck_top">
+		<origin rpy="0 0 0" xyz="0 0 0" />
+	</xacro:head_v0> -->
 </robot>

File: src/kaspar_description/urdf/kaspar_arm.xacro (robot description, xacro)
@@ -1,3 +1,28 @@
 <?xml version="1.0"?>
 <robot xmlns:xacro="http://www.ros.org/wiki/xacro">
+	<xacro:macro name="arm_v0" params="name parent *origin">
+		<xacro:mount name="${name}_mount" parent="${parent}">
+			<insert_block name="origin" />
+		</xacro:mount>
+		<xacro:drs_x01 name="${name}_0" mountTop="false" mountBottom="false" mountBack="true" mountAxel="false" parent="${name}_mount"
+			minPosition="0" maxPosition="PI" maxVelocity="1">
+			<origin xyz="0 0 0" />
+		</xacro:drs_x01>
+		<xacro:drs_x01 name="${name}_1" parent="${name}_0_axel" mountTop="false" mountBottom="true" mountBack="false" mountAxel="false"
+			minPosition="0" maxPosition="PI" maxVelocity="1">
+			<origin xyz="0 0 0" />
+		</xacro:drs_x01>
+		<xacro:drs_x01 name="${name}_2" parent="${name}_1_axel" mountTop="false" mountBottom="true" mountBack="false" mountAxel="false"
+			minPosition="0" maxPosition="PI" maxVelocity="1">
+			<origin xyz="0 0 0" />
+		</xacro:drs_x01>
+		<xacro:drs_x01 name="${name}_3" parent="${name}_2_axel" mountTop="false" mountBottom="true" mountBack="false" mountAxel="false"
+			minPosition="0" maxPosition="PI" maxVelocity="1">
+			<origin xyz="0 0 0" />
+		</xacro:drs_x01>
+		<xacro:mount name="${name}_hand" parent="${name}_3_box">
+			<origin rpy="0 0 0" xyz="0 0 0.10" />
+		</xacro:mount>
+	</xacro:macro>
+	<xacro:macro name="hand_v0" params="name parent *origin"></xacro:macro>
 </robot>

File: src/kaspar_description/urdf/kaspar_base.xacro (robot description, xacro)
@@ -2,7 +2,10 @@
 <robot xmlns:xacro="http://www.ros.org/wiki/xacro">
 	<xacro:macro name="leg_v0" params="name parent *origin">
+		<xacro:mount name="${name}_mount" parent="${parent}">
+			<insert_block name="origin" />
+		</xacro:mount>
 		<joint name="${name}_joint" type="fixed">
-			<insert_block name="origin" />
-			<parent link="${parent}_link" />
+			<origin rpy="0 0 0" xyz="0 0 0" />
+			<parent link="${name}_mount_link" />
 			<child link="${name}_link" />
 		</joint>
@@ -13,19 +16,57 @@
 			</inertial>
 			<visual>
-				<origin xyz="0 0 0.075" rpy="0 0 0" />
+				<origin xyz="0 0 0.05" rpy="0 0 0" />
 				<geometry>
-					<cylinder length="0.15" radius="0.03" />
+					<cylinder length="0.10" radius="0.03" />
 				</geometry>
-				<material name="white" />
+				<material name="trousers" />
 			</visual>
 			<collision>
-				<origin xyz="0 0 0.075" rpy="0 0 0" />
+				<origin xyz="0 0 0.05" rpy="0 0 0" />
 				<geometry>
-					<cylinder length="0.15" radius="0.03" />
+					<cylinder length="0.10" radius="0.03" />
 				</geometry>
 			</collision>
 		</link>
+		<xacro:mount name="${name}_foot" parent="${name}">
+			<origin rpy="0 0 0" xyz="0 0 0.10" />
+		</xacro:mount>
 		<gazebo reference="${name}_link">
-			<material>Gazebo/White</material>
+			<material>Gazebo/Blue</material>
+		</gazebo>
+	</xacro:macro>
+	<xacro:macro name="foot_v0" params="name parent *origin">
+		<xacro:mount name="${name}_mount" parent="${parent}">
+			<insert_block name="origin" />
+		</xacro:mount>
+		<joint name="${name}_ankle_joint" type="fixed">
+			<origin rpy="0 -1.57079 0" xyz="-0.0125 0 0.025" />
+			<parent link="${name}_mount_link" />
+			<child link="${name}_link" />
+		</joint>
+		<link name="${name}_link">
+			<inertial>
+				<mass value="0.01" />
+				<inertia ixx="0.001" ixy="0.0" ixz="0.0" iyy="0.001" iyz="0.0" izz="0.001" />
+			</inertial>
+			<visual>
+				<origin xyz="0 0 0" rpy="0 0 0" />
+				<geometry>
+					<cylinder length="0.075" radius="0.025" />
+				</geometry>
+				<material name="skin" />
+			</visual>
+			<collision>
+				<origin xyz="0 0 0" rpy="0 0 0" />
+				<geometry>
+					<cylinder length="0.075" radius="0.025" />
+				</geometry>
+			</collision>
+		</link>
+		<xacro:mount name="${name}_toe" parent="${name}">
+			<origin rpy="0 0 0" xyz="0 0 0.0375" />
+		</xacro:mount>
+		<gazebo reference="${name}_link">
+			<material>Gazebo/Yellow</material>
 		</gazebo>
 	</xacro:macro>
@@ -47,5 +88,5 @@
 					<cylinder length="0.10" radius="0.075" />
 				</geometry>
-				<material name="white" />
+				<material name="trousers" />
 			</visual>
 			<collision>
@@ -66,5 +107,5 @@
 		</xacro:mount>
 		<gazebo reference="${name}_link">
-			<material>Gazebo/White</material>
+			<material>Gazebo/Blue</material>
 		</gazebo>
 	</xacro:macro>

File: src/kaspar_description/urdf/kaspar_head.xacro (robot description, xacro)
@@ -1,4 +1,11 @@
 <?xml version="1.0"?>
 <robot xmlns:xacro="http://www.ros.org/wiki/xacro">
+	<xacro:macro name="head_v0" params="name parent *origin">
+	</xacro:macro>
+	<xacro:macro name="neck_v0" params="name parent *origin">
+		<xacro:mount name="${name}_top" parent="${name}">
+			<origin rpy="0 0 0" xyz="0 0 0.05" />
+		</xacro:mount>
+	</xacro:macro>
 	<xacro:macro name="eye" params="name parent *origin">
 		<joint name="${name}_joint" type="fixed">

File: src/kaspar_description/urdf/kaspar_mount.xacro (robot description, xacro)
@@ -9,12 +9,12 @@
 		<link name="${name}_link">
 			<inertial>
-				<origin xyz="0 0 0.0005" rpy="0 0 0" />
+				<origin xyz="0 0 0" rpy="0 0 0" />
 				<mass value="0.0001" />
 				<inertia ixx="0.001" ixy="0.0" ixz="0.0" iyy="0.001" iyz="0.0" izz="0.001" />
 			</inertial>
 			<visual>
-				<origin xyz="0 0 0.0005" rpy="0 0 0" />
+				<origin xyz="0 0 0" rpy="0 0 0" />
 				<geometry>
-					<box size="0.02 0.02 0.001" />
+					<cylinder length="0.001" radius="0.01" />
 				</geometry>
 				<material name="mount" />

File: src/kaspar_description/urdf/kaspar_torso.xacro (robot description, xacro)
@@ -2,8 +2,13 @@
 <robot xmlns:xacro="http://www.ros.org/wiki/xacro">
 	<xacro:macro name="torso_v0" params="name parent *origin">
-		<joint name="${name}_joint" type="fixed">
+		<xacro:mount name="${name}_mount" parent="${parent}">
 			<insert_block name="origin" />
-			<parent link="${parent}_link" />
+		</xacro:mount>
+		<joint name="${name}_joint" type="revolute">
+			<origin xyz="0 0 0" rpy="0 0 0" />
+			<parent link="${name}_mount_link" />
 			<child link="${name}_link" />
+			<axis xyz="0 0 1" />
+			<limit effort="0" lower="-1.5707" upper="1.5707" velocity="1" />
 		</joint>
 		<link name="${name}_link">
@@ -18,8 +23,8 @@
 					<cylinder length="0.15" radius="0.08" />
 				</geometry>
-				<material name="white" />
+				<material name="shell" />
 			</visual>
 			<collision>
-				<origin xyz="0 0 0.05" rpy="0 0 0" />
+				<origin xyz="0 0 0.08" rpy="0 0 0" />
 				<geometry>
 					<cylinder length="0.15" radius="0.08" />
@@ -28,5 +33,5 @@
 		</link>
 		<xacro:mount name="${name}_top" parent="${name}">
-			<origin rpy="0 0 0" xyz="0 0 0.15" />
+			<origin rpy="0 0 0" xyz="0 0 0.155" />
 		</xacro:mount>
 		<xacro:mount name="${name}_arm_l" parent="${name}">

File: src/kaspar_description/urdf/materials.xacro (robot description, xacro)
@@ -1,6 +1,15 @@
 <?xml version="1.0"?>
 <robot>
+	<material name="trousers">
+		<color rgba="0.0 0.0 0.8 1.0" />
+	</material>
+	<material name="shell">
+		<color rgba="1.0 1.0 1.0 0.25" />
+	</material>
 	<material name="mount">
-		<color rgba="0.08 0.08 0.08 1.0" />
+		<color rgba="0.2 0.2 0.2 0.75" />
+	</material>
+	<material name="skin">
+		<color rgba="${255/255} ${217/255} ${15/255} 0.95" />
 	</material>
 	<material name="black">
