Commit message: Rough out full urdf

File: src/herkulex/herkulex_description/urdf/drs_x01.xacro (robot description, xacro)
@@ -2,22 +2,19 @@
 <robot xmlns:controller="http://playerstage.sourceforge.net/gazebo/xmlschema/#controller" xmlns:interface="http://playerstage.sourceforge.net/gazebo/xmlschema/#interface"
 	xmlns:sensor="http://playerstage.sourceforge.net/gazebo/xmlschema/#sensor" xmlns:xacro="http://ros.org/wiki/xacro">
-	<xacro:macro name="drs_x01" params="name parent mountTop mountBottom mountBack mountAxel minPosition maxPosition maxVelocity *origin">
-		<xacro:mount name="${name}_mount" parent="${parent}">
+	<xacro:macro name="drs_x01" params="name parent mountBottom mountBack mountAxel minPosition maxPosition maxVelocity *origin">
+		<xacro:mount_point name="${name}_mount" parent="${parent}">
 			<insert_block name="origin" />
-		</xacro:mount>
-		<xacro:__drs_x01_box skipBottom="${mountBottom}" skipTop="${mountTop}" skipAxel="${mountAxel}" skipBack="${mountBack}"
+		</xacro:mount_point>
+		<xacro:__drs_x01_box skipBottom="${mountBottom}" skipAxel="${mountAxel}" skipBack="${mountBack}"
 			name="${name}" />
 		<joint name="${name}_box_joint" type="fixed">
 			<xacro:if value="${mountBack}">
-				<origin xyz="0 0 0.019" rpy="1.57079 0 -1.57079" />
+				<origin xyz="0 0 0.019" rpy="${PI / 2} 0 -${PI / 2}" />
 			</xacro:if>
 			<xacro:if value="${mountBottom}">
-				<origin xyz="0.025 0 0" rpy="0 1.57079 0" />
-			</xacro:if>
-			<xacro:if value="${mountTop}">
-				<origin xyz="-0.025 0 0" rpy="0 -1.57079 0" />
+				<origin xyz="0 0 0.025" rpy="0 ${PI / 2} 0" />
 			</xacro:if>
 			<xacro:if value="${mountAxel}">
-				<origin xyz="-0.012 0 0.019" rpy="1.57079 0 0" />
+				<origin xyz="-0.012 0 0.019" rpy="${PI / 2} 0 0" />
 			</xacro:if>
 			<xacro:if value="${mountAxel}">
@@ -30,5 +27,5 @@
 		</joint>
 		<xacro:__drs_x01_axel name="${name}" mountAxel="${mountAxel}" />
-		<joint name="${name}_axel_box_joint" type="revolute">
+		<joint name="${name}_joint" type="revolute">
 			<xacro:if value="${mountAxel}">
 				<parent link="${name}_axel_box_link" />
@@ -42,5 +39,6 @@
 			</xacro:unless>
 			<axis xyz="0 0 1" />
-			<limit effort="0" lower="-1.5707" upper="1.5707" velocity="1" />
+			<limit effort="100" velocity="${maxVelocity}" lower="${minPosition}" upper="${maxPosition}" />
+			<dynamics friction="0.01" damping="0.01" />
 		</joint>
 		<!-- Gazebo Config -->
@@ -48,8 +46,8 @@
 			<type>transmission_interface/SimpleTransmission</type>
 			<joint name="${name}_joint">
-				<hardwareInterface>PositionJointInterface</hardwareInterface>
+				<hardwareInterface>EffortJointInterface</hardwareInterface>
 			</joint>
 			<actuator name="${name}_motor">
-				<hardwareInterface>PositionJointInterface</hardwareInterface>
+				<hardwareInterface>EffortJointInterface</hardwareInterface>
 				<mechanicalReduction>1</mechanicalReduction>
 			</actuator>
@@ -62,15 +60,16 @@
 		</gazebo>
 	</xacro:macro>
-	<xacro:macro name="__drs_x01_box" params="name skipBack skipBottom skipTop skipAxel">
+	<xacro:macro name="__drs_x01_box" params="name skipBack skipBottom skipAxel">
 		<link name="${name}_box_link">
 			<visual>
-				<geometry name="x01">
-					<box size="0.050 0.038 0.032" />
+				<geometry name="x01mesh">
+					<mesh filename="package://herkulex_description/meshes/x01_box_plain.stl" scale="0.001 0.001 0.001" />
 				</geometry>
 				<material name="plastic_black" />
+				<origin rpy="${PI} 0 0" xyz="0 0 0" />
 			</visual>
 			<inertial>
-				<mass value="0.01" />
-				<inertia ixx="0.001" ixy="0.0" ixz="0.0" iyy="0.001" iyz="0.0" izz="0.001" />
+				<mass value="0.001" />
+				<inertia ixx="0.01" ixy="0.0" ixz="0.0" iyy="0.01" iyz="0.0" izz="0.01" />
 			</inertial>
 			<collision>
@@ -81,32 +80,28 @@
 		</link>
 		<xacro:unless value="${skipBack}">
-			<xacro:mount name="${name}_box_back" parent="${name}_box">
-				<origin xyz="0 0.019 0" rpy="1.57079 0 0" />
-			</xacro:mount>
+			<xacro:mount_point name="${name}_box_back" parent="${name}_box">
+				<origin xyz="0 -0.019 0" rpy="${PI / 2} 0 0" />
+			</xacro:mount_point>
 		</xacro:unless>
 		<xacro:unless value="${skipBottom}">
-			<xacro:mount name="${name}_box_bottom" parent="${name}_box">
-				<origin xyz="0.025 0 0" rpy="0 1.57079 0" />
-			</xacro:mount>
-		</xacro:unless>
-		<xacro:unless value="${skipTop}">
-			<xacro:mount name="${name}_box_top" parent="${name}_box">
-				<origin xyz="-0.025 0 0" rpy="0 -1.57079 0" />
-			</xacro:mount>
+			<xacro:mount_point name="${name}_box_bottom" parent="${name}_box">
+				<origin xyz="0.025 0 0" rpy="0 ${PI / 2} 0" />
+			</xacro:mount_point>
 		</xacro:unless>
 		<xacro:unless value="${skipAxel}">
-			<xacro:mount name="${name}_box_axel" parent="${name}_box">
-				<origin xyz="-0.012 0.019 0" rpy="1.57075 0 3.14159" />
-			</xacro:mount>
+			<xacro:mount_point name="${name}_box_axel" parent="${name}_box">
+				<origin xyz="-0.012 0.019 0" rpy="${PI / 2} 0 ${PI}" />
+			</xacro:mount_point>
 		</xacro:unless>
 		<xacro:if value="${skipAxel}">
 			<link name="${name}_box_axel_link">
-			<visual>
-				<origin xyz="0 0 0" rpy="0 0 0" />
-				<geometry>
-					<cylinder length="0.001" radius="0.01" />
-				</geometry>
-				<material name="orange" />
-			</visual></link>
+				<visual>
+					<origin xyz="0 0 0" rpy="0 0 0" />
+					<geometry>
+						<cylinder length="0.001" radius="0.01" />
+					</geometry>
+					<material name="orange" />
+				</visual>
+			</link>
 		</xacro:if>
 	</xacro:macro>
@@ -130,61 +125,18 @@
 		</link>
 		<xacro:if value="${mountAxel}">
-			<xacro:mount name="${name}_axel" parent="${name}_mount">
+			<xacro:mount_point name="${name}_axel" parent="${name}_mount">
 				<origin xyz="0 0 -0.0025" rpy="0 0 0" />
-			</xacro:mount>
+			</xacro:mount_point>
 			<joint name="${name}_axel0_joint" type="fixed">
 				<parent link="${name}_axel_link" />
 				<child link="${name}_axel_box_link" />
-				<origin xyz="0 0 0" rpy="0 0 1.57079" />
+				<origin xyz="0 0 0" rpy="0 0 ${PI / 2}" />
 			</joint>
 		</xacro:if>
 		<xacro:unless value="${mountAxel}">
-			<xacro:mount name="${name}_axel" parent="${name}_axel_box">
-				<origin xyz="0 0 0.0025" rpy="0 0 1.57079" />
-			</xacro:mount>
+			<xacro:mount_point name="${name}_axel" parent="${name}_axel_box">
+				<origin xyz="0 0 0.0025" rpy="0 0 ${PI / 2}" />
+			</xacro:mount_point>
 		</xacro:unless>
 	</xacro:macro>
-	<xacro:macro name="drs_x01_axel" params="name parent minPosition maxPosition maxVelocity *origin">
-		<xacro:mount name="${name}_mount" parent="${parent}">
-			<insert_block name="origin" />
-		</xacro:mount>
-		<xacro:__drs_x01_box skip="" name="${name}" />
-		<xacro:__drs_x01_axel name="${name}" />
-		<joint name="${name}_axel_joint" type="fixed">
-			<origin rpy="0 0 0" xyz="0 0 0" />
-			<parent link="${name}_mount_link" />
-			<child link="${name}_axel_link" />
-		</joint>
-		<joint name="${name}_joint" type="fixed">
-			<parent link="${name}_axel_link" />
-			<child link="${name}_box_axel0_link" />
-			<origin xyz="0 0 -0.001" rpy="0 0 0" />
-			<axis xyz="0 0 1" />
-			<limit effort="0" lower="-1.5707" upper="1.5707" velocity="1" />
-		</joint>
-		<link name="${name}_box_axel_link">
-		</link>
-		<joint name="${name}_axel_joint" type="fixed">
-			<parent link="${name}_box_axel_link" />
-			<child link="${name}_box_link" />
-			<origin xyz="-0.012 0 0.025" rpy="1.57075 0 3.14159" />
-		</joint>
-		<!-- Gazebo Config -->
-		<transmission name="${name}_trans">
-			<type>transmission_interface/SimpleTransmission</type>
-			<joint name="${name}_joint">
-				<hardwareInterface>PositionJointInterface</hardwareInterface>
-			</joint>
-			<actuator name="${name}_motor">
-				<hardwareInterface>PositionJointInterface</hardwareInterface>
-				<mechanicalReduction>1</mechanicalReduction>
-			</actuator>
-		</transmission>
-		<gazebo reference="${name}_box_link">
-			<material>Gazebo/FlatBlack</material>
-		</gazebo>
-		<gazebo reference="${name}_box_axel_link">
-			<material>Gazebo/White</material>
-		</gazebo>
-	</xacro:macro>
 </robot>

File: src/herkulex/herkulex_description/urdf/mount.xacro (robot description, xacro)
@@ -1,37 +1,28 @@
-<?xml version="1.0" encoding="UTF-8"?>
-<robot
-	xmlns:controller="http://playerstage.sourceforge.net/gazebo/xmlschema/#controller"
-	xmlns:interface="http://playerstage.sourceforge.net/gazebo/xmlschema/#interface"
-	xmlns:sensor="http://playerstage.sourceforge.net/gazebo/xmlschema/#sensor"
-	xmlns:xacro="http://ros.org/wiki/xacro">
-	<xacro:macro name="fp04_02" params="name parent">
+<?xml version="1.0"?>
+<robot xmlns:xacro="http://www.ros.org/wiki/xacro">
+	<xacro:macro name="mount_v0" params="name parent *origin">
+		<xacro:mount_point name="${name}_mount" parent="${parent}">
+			<insert_block name="origin" />
+		</xacro:mount_point>
 		<link name="${name}_mesh_link">
 			<visual>
-				<geometry name="fp04_02mesh">
-					<mesh filename="package://dynamixel_description/meshes/F2.stl" scale="0.001 0.001 0.001" />
+				<geometry name="mount_mesh">
+					<mesh filename="package://herkulex_description/meshes/mount.stl" scale="0.001 0.001 0.001" />
 				</geometry>
-				<material name="plastic_green">
-					<color rgba="0.1 0.8 0.3 1" />
-				</material>
-				<origin rpy="-1.57075 0 1.57075" xyz="0 0 0.0" />
+				<material name="plastic_green" />
 			</visual>
 			<inertial>
 				<mass value="0.005" />
-				<inertia ixx="0.001" ixy="0.0" ixz="0.0" iyy="0.001" iyz="0.0"
-					izz="0.001" />
-				<origin rpy="0 0 0" xyz="0 0 0.0025" />
+				<inertia ixx="0.001" ixy="0.0" ixz="0.0" iyy="0.001" iyz="0.0" izz="0.001" />
 			</inertial>
 		</link>
-		<link name="${name}_link"></link>
-		<joint name="${name}_joint" type="fixed">
-			<parent link="${name}_mesh_link" />
-			<child link="${name}_link" />
-			<origin xyz="0 0 0.027" />
+		<joint name="${name}_mesh_joint" type="fixed">
+			<parent link="${name}_mount_link" />
+			<child link="${name}_mesh_link" />
+			<origin rpy="${PI} 0 0" xyz="0 0 -0.0205" />
 		</joint>
-		<joint name="${name}_mesh_joint" type="fixed">
-			<parent link="${parent}_link" />
-			<child link="${name}_mesh_link" />
-			<origin xyz="-0.015 0 0" />
-		</joint>
+		<xacro:mount_point name="${name}" parent="${name}_mesh">
+			<origin xyz="0 -0.027 0" rpy="${PI / 2} 0 0" />
+		</xacro:mount_point>
 		<gazebo reference="${name}_mesh_link">
 			<material>Gazebo/Green</material>

File: src/kaspar_description/urdf/kaspar.xacro (robot description, xacro)
@@ -1,7 +1,6 @@
 <?xml version="1.0"?>
 <robot name="kaspar" xmlns:xacro="http://www.ros.org/wiki/xacro">
-	<!-- Constants for robot dimensions -->
+	<!-- Constants -->
 	<xacro:property name="PI" value="3.1415926535897931" />
-	<xacro:property name="mass" value="10" />
 	<!-- Import joint description -->
 	<xacro:include filename="$(find herkulex_description)/urdf/drs_x01.xacro" />
@@ -37,12 +36,11 @@
 		<origin rpy="0 0 0" xyz="0 0 0" />
 	</xacro:arm_v0>
-	<!--
-	<xacro:hand_v0 name="hand_r" parent="torso_arm_r_hand">
+	<xacro:hand_v0 name="hand_r" parent="arm_r_hand">
 		<origin rpy="0 0 0" xyz="0 0 0" />
 	</xacro:hand_v0>
 	<xacro:arm_v0 name="arm_l" parent="torso_arm_l">
-		<origin rpy="0 0 0" xyz="0 0 0" />
+		<origin rpy="0 0 ${PI}" xyz="0 0 0" />
 	</xacro:arm_v0>
-	<xacro:hand_v0 name="hand_l" parent="torso_arm_l_hand">
+	<xacro:hand_v0 name="hand_l" parent="arm_l_hand">
 		<origin rpy="0 0 0" xyz="0 0 0" />
 	</xacro:hand_v0>
@@ -52,4 +50,11 @@
 	<xacro:head_v0 name="head" parent="neck_top">
 		<origin rpy="0 0 0" xyz="0 0 0" />
-	</xacro:head_v0> -->
+	</xacro:head_v0>
+  <!-- ros_control plugin -->
+  <gazebo>
+    <plugin name="gazebo_ros_control" filename="libgazebo_ros_control.so">
+      <robotNamespace>/kaspar</robotNamespace>
+      <robotSimType>gazebo_ros_control/DefaultRobotHWSim</robotSimType>
+    </plugin>
+  </gazebo>
 </robot>

File: src/kaspar_description/urdf/kaspar_arm.xacro (robot description, xacro)
@@ -1,28 +1,62 @@
 <?xml version="1.0"?>
 <robot xmlns:xacro="http://www.ros.org/wiki/xacro">
+	<xacro:macro name="hand_v0" params="name parent *origin">
+		<xacro:mount_point name="${name}_mount" parent="${parent}">
+			<insert_block name="origin" />
+		</xacro:mount_point>
+		<joint name="${name}_wrist_joint" type="fixed">
+			<origin rpy="0 0 0" xyz="0 0 0.0275" />
+			<parent link="${name}_mount_link" />
+			<child link="${name}_link" />
+		</joint>
+		<link name="${name}_link">
+			<inertial>
+				<mass value="0.25" />
+				<inertia ixx="0.25" ixy="0.0" ixz="0.0" iyy="0.25" iyz="0.0" izz="0.25" />
+			</inertial>
+			<visual>
+				<origin xyz="0 0 0" rpy="0 0 0" />
+				<geometry>
+					<cylinder length="0.055" radius="0.015" />
+				</geometry>
+				<material name="skin" />
+			</visual>
+			<collision>
+				<origin xyz="0 0 0" rpy="0 0 0" />
+				<geometry>
+					<cylinder length="0.055" radius="0.015" />
+				</geometry>
+			</collision>
+		</link>
+		<xacro:mount_point name="${name}_fingers" parent="${name}">
+			<origin rpy="0 0 0" xyz="0 0 0.0275" />
+		</xacro:mount_point>
+		<gazebo reference="${name}_link">
+			<material>Gazebo/Yellow</material>
+		</gazebo>
+	</xacro:macro>
 	<xacro:macro name="arm_v0" params="name parent *origin">
-		<xacro:mount name="${name}_mount" parent="${parent}">
+		<xacro:mount_point name="${name}_mount" parent="${parent}">
 			<insert_block name="origin" />
-		</xacro:mount>
-		<xacro:drs_x01 name="${name}_0" mountTop="false" mountBottom="false" mountBack="true" mountAxel="false" parent="${name}_mount"
-			minPosition="0" maxPosition="PI" maxVelocity="1">
+		</xacro:mount_point>
+		<xacro:drs_x01 name="${name}_0" mountBottom="false" mountBack="true" mountAxel="false" parent="${name}_mount" minPosition="${PI}"
+			maxPosition="${PI}" maxVelocity="1">
 			<origin xyz="0 0 0" />
 		</xacro:drs_x01>
-		<xacro:drs_x01 name="${name}_1" parent="${name}_0_axel" mountTop="false" mountBottom="true" mountBack="false" mountAxel="false"
-			minPosition="0" maxPosition="PI" maxVelocity="1">
+		<xacro:drs_x01 name="${name}_1" parent="${name}_0_axel" mountBottom="true" mountBack="false" mountAxel="false" minPosition="${PI}"
+			maxPosition="${PI}" maxVelocity="1">
 			<origin xyz="0 0 0" />
 		</xacro:drs_x01>
-		<xacro:drs_x01 name="${name}_2" parent="${name}_1_axel" mountTop="false" mountBottom="true" mountBack="false" mountAxel="false"
-			minPosition="0" maxPosition="PI" maxVelocity="1">
+		<xacro:drs_x01 name="${name}_2" parent="${name}_1_axel" mountBottom="true" mountBack="false" mountAxel="false" minPosition="${PI}"
+			maxPosition="${PI}" maxVelocity="1">
 			<origin xyz="0 0 0" />
 		</xacro:drs_x01>
-		<xacro:drs_x01 name="${name}_3" parent="${name}_2_axel" mountTop="false" mountBottom="true" mountBack="false" mountAxel="false"
-			minPosition="0" maxPosition="PI" maxVelocity="1">
+		<xacro:drs_x01 name="${name}_3" parent="${name}_2_axel" mountBottom="true" mountBack="false" mountAxel="false" minPosition="${PI}"
+			maxPosition="${PI}" maxVelocity="1">
 			<origin xyz="0 0 0" />
 		</xacro:drs_x01>
-		<xacro:mount name="${name}_hand" parent="${name}_3_box">
-			<origin rpy="0 0 0" xyz="0 0 0.10" />
-		</xacro:mount>
+		<xacro:mount_point name="${name}_hand" parent="${name}_3_axel">
+			<origin rpy="0 0 0" xyz="0 0 0" />
+		</xacro:mount_point>
 	</xacro:macro>
-	<xacro:macro name="hand_v0" params="name parent *origin"></xacro:macro>
 </robot>

File: src/kaspar_description/urdf/kaspar_base.xacro (robot description, xacro)
@@ -2,7 +2,7 @@
 <robot xmlns:xacro="http://www.ros.org/wiki/xacro">
 	<xacro:macro name="leg_v0" params="name parent *origin">
-		<xacro:mount name="${name}_mount" parent="${parent}">
+		<xacro:mount_point name="${name}_mount" parent="${parent}">
 			<insert_block name="origin" />
-		</xacro:mount>
+		</xacro:mount_point>
 		<joint name="${name}_joint" type="fixed">
 			<origin rpy="0 0 0" xyz="0 0 0" />
@@ -12,6 +12,6 @@
 		<link name="${name}_link">
 			<inertial>
-				<mass value="0.1" />
-				<inertia ixx="0.001" ixy="0.0" ixz="0.0" iyy="0.001" iyz="0.0" izz="0.001" />
+				<mass value="1" />
+				<inertia ixx="1.0" ixy="0.0" ixz="0.0" iyy="1.0" iyz="0.0" izz="1.0" />
 			</inertial>
 			<visual>
@@ -29,7 +29,7 @@
 			</collision>
 		</link>
-		<xacro:mount name="${name}_foot" parent="${name}">
+		<xacro:mount_point name="${name}_foot" parent="${name}">
 			<origin rpy="0 0 0" xyz="0 0 0.10" />
-		</xacro:mount>
+		</xacro:mount_point>
 		<gazebo reference="${name}_link">
 			<material>Gazebo/Blue</material>
@@ -37,9 +37,9 @@
 	</xacro:macro>
 	<xacro:macro name="foot_v0" params="name parent *origin">
-		<xacro:mount name="${name}_mount" parent="${parent}">
+		<xacro:mount_point name="${name}_mount" parent="${parent}">
 			<insert_block name="origin" />
-		</xacro:mount>
+		</xacro:mount_point>
 		<joint name="${name}_ankle_joint" type="fixed">
-			<origin rpy="0 -1.57079 0" xyz="-0.0125 0 0.025" />
+			<origin rpy="0 -${PI / 2} 0" xyz="-0.0125 0 0.025" />
 			<parent link="${name}_mount_link" />
 			<child link="${name}_link" />
@@ -47,6 +47,6 @@
 		<link name="${name}_link">
 			<inertial>
-				<mass value="0.01" />
-				<inertia ixx="0.001" ixy="0.0" ixz="0.0" iyy="0.001" iyz="0.0" izz="0.001" />
+				<mass value="0.5" />
+				<inertia ixx="0.5" ixy="0.0" ixz="0.0" iyy="0.5" iyz="0.0" izz="0.5" />
 			</inertial>
 			<visual>
@@ -64,7 +64,7 @@
 			</collision>
 		</link>
-		<xacro:mount name="${name}_toe" parent="${name}">
+		<xacro:mount_point name="${name}_toe" parent="${name}">
 			<origin rpy="0 0 0" xyz="0 0 0.0375" />
-		</xacro:mount>
+		</xacro:mount_point>
 		<gazebo reference="${name}_link">
 			<material>Gazebo/Yellow</material>
@@ -79,7 +79,7 @@
 		<link name="${name}_link">
 			<inertial>
+				<origin xyz="0 0 0.05" rpy="0 0 0" />
 				<mass value="5" />
-				<origin xyz="0 0 0.05" rpy="0 0 0" />
-				<inertia ixx="0.001" ixy="0.0" ixz="0.0" iyy="0.001" iyz="0.0" izz="0.001" />
+				<inertia ixx="5.0" ixy="0.0" ixz="0.0" iyy="5.0" iyz="0.0" izz="5.0" />
 			</inertial>
 			<visual>
@@ -97,13 +97,13 @@
 			</collision>
 		</link>
-		<xacro:mount name="${name}_top" parent="${name}">
+		<xacro:mount_point name="${name}_top" parent="${name}">
 			<origin rpy="0 0 0" xyz="0 0 0.10" />
-		</xacro:mount>
-		<xacro:mount name="${name}_leg_l" parent="${name}">
+		</xacro:mount_point>
+		<xacro:mount_point name="${name}_leg_l" parent="${name}">
 			<origin rpy="0 ${PI / 2} ${PI / 4}" xyz="0.053033009 0.053033009 0.03" />
-		</xacro:mount>
-		<xacro:mount name="${name}_leg_r" parent="${name}">
+		</xacro:mount_point>
+		<xacro:mount_point name="${name}_leg_r" parent="${name}">
 			<origin rpy="0 ${PI / 2} -${PI / 4}" xyz="0.053033009 -0.053033009 0.03" />
-		</xacro:mount>
+		</xacro:mount_point>
 		<gazebo reference="${name}_link">
 			<material>Gazebo/Blue</material>

File: src/kaspar_description/urdf/kaspar_head.xacro (robot description, xacro)
@@ -2,84 +2,47 @@
 <robot xmlns:xacro="http://www.ros.org/wiki/xacro">
 	<xacro:macro name="head_v0" params="name parent *origin">
-	</xacro:macro>
-	<xacro:macro name="neck_v0" params="name parent *origin">
-		<xacro:mount name="${name}_top" parent="${name}">
-			<origin rpy="0 0 0" xyz="0 0 0.05" />
-		</xacro:mount>
-	</xacro:macro>
-	<xacro:macro name="eye" params="name parent *origin">
+		<xacro:mount_point name="${name}_mount" parent="${parent}">
+			<insert_block name="origin" />
+		</xacro:mount_point>
 		<joint name="${name}_joint" type="fixed">
-			<insert_block name="origin" />
-			<parent link="${parent}_link" />
+			<origin rpy="0 0 0" xyz="0 0 0.09" />
+			<parent link="${name}_mount_link" />
 			<child link="${name}_link" />
 		</joint>
 		<link name="${name}_link">
-			<inertial>
-				<mass value="0.01" />
-				<inertia ixx="0.001" ixy="0.0" ixz="0.0" iyy="0.001" iyz="0.0" izz="0.001" />
-			</inertial>
 			<visual>
-				<origin rpy="0 1.5707 0" />
 				<geometry>
-					<cylinder length="0.015" radius="0.03" />
+					<sphere radius="0.08" />
 				</geometry>
-				<material name="white">
-					<color rgba="0.98 0.98 0.90 1.0" />
-				</material>
+				<material name="skin" />
 			</visual>
 			<collision>
-				<origin rpy="0 1.5707 0" />
 				<geometry>
-					<cylinder length="0.015" radius="0.03" />
+					<sphere radius="0.08" />
 				</geometry>
 			</collision>
 		</link>
+		<xacro:mount_point name="${name}_top" parent="${name}">
+			<origin xyz="0 0 0.08" rpy="0 0 0" />
+		</xacro:mount_point>
 		<gazebo reference="${name}_link">
-			<material>Gazebo/White</material>
+			<material>Gazebo/Yellow</material>
 		</gazebo>
 	</xacro:macro>
-	<xacro:macro name="head" params="name parent *origin">
-		<joint name="${name}_mount_joint" type="fixed">
+	<xacro:macro name="neck_v0" params="name parent *origin">
+		<xacro:mount_point name="${name}_mount" parent="${parent}">
 			<insert_block name="origin" />
-			<parent link="${parent}_link" />
-			<child link="${name}_mount_link" />
-		</joint>
-		<link name="${name}_mount_link"></link>
-		<joint name="${name}_joint" type="fixed">
-			<parent link="${name}_mount_link" />
-			<child link="${name}_link" />
-			<origin rpy="0 0 0 " xyz="0 0 -0.0475" />
-		</joint>
-		<link name="${name}_link">
-			<inertial>
-				<mass value="0.1" />
-				<inertia ixx="0.001" ixy="0.0" ixz="0.0" iyy="0.001" iyz="0.0" izz="0.001" />
-			</inertial>
-			<visual>
-				<geometry>
-					<cylinder length="0.10" radius="0.11" />
-				</geometry>
-				<material name="grey">
-					<color rgba="0.5 0.5 0.5 1.0" />
-				</material>
-			</visual>
-			<collision>
-				<geometry>
-					<cylinder length="0.10" radius="0.11" />
-				</geometry>
-			</collision>
-		</link>
-		<gazebo reference="${name}_link">
-			<material>Gazebo/Grey</material>
-		</gazebo>
-		<xacro:eye name="eye_r" parent="${name}">
-			<origin rpy="0 0 -0.23" xyz="0.12 -0.06 0" />
-		</xacro:eye>
-		<xacro:eye name="eye_l" parent="${name}">
-			<origin rpy="0 0 0.23" xyz="0.12 0.06 0" />
-		</xacro:eye>
-		<xacro:simple_camera name="camera" parent="${name}">
-			<origin rpy="0 0 0" xyz="0.11 0.00 -0.02" />
-		</xacro:simple_camera>
+		</xacro:mount_point>
+		<xacro:drs_x01 name="${name}_0" mountBottom="false" mountBack="true" mountAxel="false" parent="${name}_mount" minPosition="${PI}"
+			maxPosition="${PI}" maxVelocity="1">
+			<origin xyz="0 0 0" />
+		</xacro:drs_x01>
+		<xacro:drs_x01 name="${name}_1" parent="${name}_0_axel" mountBottom="true" mountBack="false" mountAxel="false" minPosition="${PI}"
+			maxPosition="${PI}" maxVelocity="1">
+			<origin xyz="0 0 0" rpy="0 0 ${PI}" />
+		</xacro:drs_x01>
+		<xacro:mount_v0 name="${name}_top" parent="${name}_1_axel">
+			<origin rpy="0 0 0" xyz="0 0 0" />
+		</xacro:mount_v0>
 	</xacro:macro>
 </robot>

File: src/kaspar_description/urdf/kaspar_mount.xacro (robot description, xacro)
@@ -1,5 +1,5 @@
 <?xml version="1.0"?>
 <robot xmlns:xacro="http://www.ros.org/wiki/xacro">
-	<xacro:macro name="mount" params="name parent *origin">
+	<xacro:macro name="mount_point" params="name parent *origin">
 		<joint name="${name}_joint" type="fixed">
 			<insert_block name="origin" />
