Commit message: Rough out full urdf

File: src/kaspar_description/urdf/kaspar_torso.xacro (robot description, xacro)
@@ -2,7 +2,7 @@
 <robot xmlns:xacro="http://www.ros.org/wiki/xacro">
 	<xacro:macro name="torso_v0" params="name parent *origin">
-		<xacro:mount name="${name}_mount" parent="${parent}">
+		<xacro:mount_point name="${name}_mount" parent="${parent}">
 			<insert_block name="origin" />
-		</xacro:mount>
+		</xacro:mount_point>
 		<joint name="${name}_joint" type="revolute">
 			<origin xyz="0 0 0" rpy="0 0 0" />
@@ -11,10 +11,11 @@
 			<axis xyz="0 0 1" />
 			<limit effort="0" lower="-1.5707" upper="1.5707" velocity="1" />
+			<dynamics friction="0.01" damping="0.01" />
 		</joint>
 		<link name="${name}_link">
 			<inertial>
-				<mass value="5" />
 				<origin xyz="0 0 0.08" rpy="0 0 0" />
-				<inertia ixx="0.001" ixy="0.0" ixz="0.0" iyy="0.001" iyz="0.0" izz="0.001" />
+				<mass value="0.001" />
+				<inertia ixx="0.01" ixy="0.0" ixz="0.0" iyy="0.01" iyz="0.0" izz="0.01" />
 			</inertial>
 			<visual>
@@ -32,13 +33,24 @@
 			</collision>
 		</link>
-		<xacro:mount name="${name}_top" parent="${name}">
+		<xacro:mount_point name="${name}_top" parent="${name}">
 			<origin rpy="0 0 0" xyz="0 0 0.155" />
-		</xacro:mount>
-		<xacro:mount name="${name}_arm_l" parent="${name}">
-			<origin rpy="-1.57079 0 0" xyz="0 0.08 0.12" />
-		</xacro:mount>
-		<xacro:mount name="${name}_arm_r" parent="${name}">
-			<origin rpy="1.57079 0 0" xyz="0 -0.08 0.12" />
-		</xacro:mount>
+		</xacro:mount_point>
+		<xacro:mount_point name="${name}_arm_l" parent="${name}">
+			<origin rpy="-${PI / 2} 0 0" xyz="0 0.08 0.12" />
+		</xacro:mount_point>
+		<xacro:mount_point name="${name}_arm_r" parent="${name}">
+			<origin rpy="${PI / 2} 0 0" xyz="0 -0.08 0.12" />
+		</xacro:mount_point>
+		<!-- Gazebo Config -->
+		<transmission name="${name}_trans">
+			<type>transmission_interface/SimpleTransmission</type>
+			<joint name="${name}_joint">
+				<hardwareInterface>EffortJointInterface</hardwareInterface>
+			</joint>
+			<actuator name="${name}_motor">
+				<hardwareInterface>EffortJointInterface</hardwareInterface>
+				<mechanicalReduction>1</mechanicalReduction>
+			</actuator>
+		</transmission>
 		<gazebo reference="${name}_link">
 			<material>Gazebo/White</material>

File: src/kaspar_description/urdf/materials.xacro (robot description, xacro)
@@ -12,4 +12,7 @@
 	<material name="skin">
 		<color rgba="${255/255} ${217/255} ${15/255} 0.95" />
+	</material>
+	<material name="plastic_green">
+		<color rgba="0.1 0.8 0.3 1" />
 	</material>
 	<material name="black">

Commit message: Fixes for inverted mount

File: src/herkulex/herkulex_description/urdf/drs_x01.xacro (robot description, xacro)
@@ -1,22 +1,26 @@
 <?xml version="1.0" encoding="UTF-8"?>
-<robot xmlns:controller="http://playerstage.sourceforge.net/gazebo/xmlschema/#controller" xmlns:interface="http://playerstage.sourceforge.net/gazebo/xmlschema/#interface"
-	xmlns:sensor="http://playerstage.sourceforge.net/gazebo/xmlschema/#sensor" xmlns:xacro="http://ros.org/wiki/xacro">
-	<xacro:macro name="drs_x01" params="name parent mountBottom mountBack mountAxel minPosition maxPosition maxVelocity *origin">
+<robot xmlns:xacro="http://ros.org/wiki/xacro">
+	<xacro:macro name="drs_x01" params="name parent mountBottom mountBack mountLeft mountRight mountAxel minPosition maxPosition maxVelocity *origin">
 		<xacro:mount_point name="${name}_mount" parent="${parent}">
 			<insert_block name="origin" />
 		</xacro:mount_point>
-		<xacro:__drs_x01_box skipBottom="${mountBottom}" skipAxel="${mountAxel}" skipBack="${mountBack}"
-			name="${name}" />
+		<!-- TODO: Jade would make this much easier, as string comparison functions are possible. i.e. "${mount=='bottom'}" -->
+		<xacro:__drs_x01_box skipBottom="${mountBottom}" skipAxel="${mountAxel}" skipBack="${mountBack}" skipLeft="${mountLeft}"
+			skipRight="${mountRight}" name="${name}" />
 		<joint name="${name}_box_joint" type="fixed">
 			<xacro:if value="${mountBack}">
-				<origin xyz="0 0 0.019" rpy="${PI / 2} 0 -${PI / 2}" />
+				<origin xyz="0.008 0 0.019" rpy="${PI / 2} 0 0" />
 			</xacro:if>
 			<xacro:if value="${mountBottom}">
 				<origin xyz="0 0 0.025" rpy="0 ${PI / 2} 0" />
 			</xacro:if>
-			<xacro:if value="${mountAxel}">
-				<origin xyz="-0.012 0 0.019" rpy="${PI / 2} 0 0" />
+			<xacro:if value="${mountLeft}">
+				<origin xyz="0 -0.007 0.016" rpy="${PI} 0 ${PI / 2}" />
+			</xacro:if>
+			<xacro:if value="${mountRight}">
+				<origin xyz="0 0.007 0.016" rpy="0 0 -${PI / 2}" />
 			</xacro:if>
 			<xacro:if value="${mountAxel}">
+				<origin xyz="0.0125 0 0.019" rpy="-${PI / 2} 0 0" />
 				<parent link="${name}_box_axel_link" />
 			</xacro:if>
@@ -60,5 +64,5 @@
 		</gazebo>
 	</xacro:macro>
-	<xacro:macro name="__drs_x01_box" params="name skipBack skipBottom skipAxel">
+	<xacro:macro name="__drs_x01_box" params="name skipBack skipBottom skipLeft skipRight skipAxel">
 		<link name="${name}_box_link">
 			<visual>
@@ -81,5 +85,5 @@
 		<xacro:unless value="${skipBack}">
 			<xacro:mount_point name="${name}_box_back" parent="${name}_box">
-				<origin xyz="0 -0.019 0" rpy="${PI / 2} 0 0" />
+				<origin xyz="0.007 -0.019 0" rpy="${PI / 2} 0 0" />
 			</xacro:mount_point>
 		</xacro:unless>
@@ -89,7 +93,17 @@
 			</xacro:mount_point>
 		</xacro:unless>
+		<xacro:unless value="${skipLeft}">
+			<xacro:mount_point name="${name}_box_left" parent="${name}_box">
+				<origin xyz="0.007 0 0.016" rpy="0 0 0" />
+			</xacro:mount_point>
+		</xacro:unless>
+		<xacro:unless value="${skipRight}">
+			<xacro:mount_point name="${name}_box_right" parent="${name}_box">
+				<origin xyz="0.007 0 -0.016" rpy="-${PI} 0 0" />
+			</xacro:mount_point>
+		</xacro:unless>
 		<xacro:unless value="${skipAxel}">
 			<xacro:mount_point name="${name}_box_axel" parent="${name}_box">
-				<origin xyz="-0.012 0.019 0" rpy="${PI / 2} 0 ${PI}" />
+				<origin xyz="-0.0125 0.019 0" rpy="${PI / 2} 0 ${PI}" />
 			</xacro:mount_point>
 		</xacro:unless>
@@ -126,10 +140,10 @@
 		<xacro:if value="${mountAxel}">
 			<xacro:mount_point name="${name}_axel" parent="${name}_mount">
-				<origin xyz="0 0 -0.0025" rpy="0 0 0" />
+				<origin xyz="0 0 0.005" rpy="0 0 0" />
 			</xacro:mount_point>
 			<joint name="${name}_axel0_joint" type="fixed">
 				<parent link="${name}_axel_link" />
 				<child link="${name}_axel_box_link" />
-				<origin xyz="0 0 0" rpy="0 0 ${PI / 2}" />
+				<origin xyz="0 0 -0.0025" rpy="0 0 ${PI / 2}" />
 			</joint>
 		</xacro:if>

File: src/herkulex/herkulex_description/urdf/mount.xacro (robot description, xacro)
@@ -1,5 +1,5 @@
 <?xml version="1.0"?>
 <robot xmlns:xacro="http://www.ros.org/wiki/xacro">
-	<xacro:macro name="mount_v0" params="name parent *origin">
+	<xacro:macro name="mount_v0" params="name invert parent *origin">
 		<xacro:mount_point name="${name}_mount" parent="${parent}">
 			<insert_block name="origin" />
@@ -20,8 +20,18 @@
 			<parent link="${name}_mount_link" />
 			<child link="${name}_mesh_link" />
-			<origin rpy="${PI} 0 0" xyz="0 0 -0.0205" />
+			<xacro:unless value="${invert}">
+				<origin rpy="${PI} 0 0" xyz="0 0 -0.0205" />
+			</xacro:unless>
+			<xacro:if value="${invert}">
+				<origin rpy="${PI / 2} 0 0" xyz="0 0 0.027" />
+			</xacro:if>
 		</joint>
 		<xacro:mount_point name="${name}" parent="${name}_mesh">
-			<origin xyz="0 -0.027 0" rpy="${PI / 2} 0 0" />
+			<xacro:unless value="${invert}">
+				<origin xyz="0 -0.027 0" rpy="${PI / 2} 0 0" />
+			</xacro:unless>
+			<xacro:if value="${invert}">
+				<origin xyz="0 0 0.0205" rpy="0 -${PI} 0" />
+			</xacro:if>
 		</xacro:mount_point>
 		<gazebo reference="${name}_mesh_link">

File: src/kaspar_description/urdf/kaspar.xacro (robot description, xacro)
@@ -1,6 +1,4 @@
 <?xml version="1.0"?>
 <robot name="kaspar" xmlns:xacro="http://www.ros.org/wiki/xacro">
-	<!-- Constants -->
-	<xacro:property name="PI" value="3.1415926535897931" />
 	<!-- Import joint description -->
 	<xacro:include filename="$(find herkulex_description)/urdf/drs_x01.xacro" />
@@ -13,4 +11,7 @@
 	<xacro:include filename="$(find kaspar_description)/urdf/kaspar_mount.xacro" />
 	<xacro:include filename="$(find kaspar_description)/urdf/materials.xacro" />
+	<!-- Constants -->
+	<xacro:property name="PI" value="3.1415926535897931" />
+	<xacro:property name="VISIBLE_MOUNTS" value="true" />
 	<!-- Used for fixing robot in the world -->
 	<link name="world_link" />
@@ -51,10 +52,10 @@
 		<origin rpy="0 0 0" xyz="0 0 0" />
 	</xacro:head_v0>
-  <!-- ros_control plugin -->
-  <gazebo>
-    <plugin name="gazebo_ros_control" filename="libgazebo_ros_control.so">
-      <robotNamespace>/kaspar</robotNamespace>
-      <robotSimType>gazebo_ros_control/DefaultRobotHWSim</robotSimType>
-    </plugin>
-  </gazebo>
+	<!-- ros_control plugin -->
+	<gazebo>
+		<plugin name="gazebo_ros_control" filename="libgazebo_ros_control.so">
+			<robotNamespace>/kaspar</robotNamespace>
+			<robotSimType>gazebo_ros_control/DefaultRobotHWSim</robotSimType>
+		</plugin>
+	</gazebo>
 </robot>

File: src/kaspar_description/urdf/kaspar_arm.xacro (robot description, xacro)
@@ -40,18 +40,21 @@
 			<insert_block name="origin" />
 		</xacro:mount_point>
-		<xacro:drs_x01 name="${name}_0" mountBottom="false" mountBack="true" mountAxel="false" parent="${name}_mount" minPosition="${PI}"
-			maxPosition="${PI}" maxVelocity="1">
+		<xacro:drs_x01 name="${name}_0" parent="${name}_mount" mountBottom="false" mountBack="true" mountLeft="false" mountRight="false"
+			mountAxel="false" minPosition="${PI}" maxPosition="${PI}" maxVelocity="1">
 			<origin xyz="0 0 0" />
 		</xacro:drs_x01>
-		<xacro:drs_x01 name="${name}_1" parent="${name}_0_axel" mountBottom="true" mountBack="false" mountAxel="false" minPosition="${PI}"
-			maxPosition="${PI}" maxVelocity="1">
+		<xacro:mount_v0 name="${name}_0_joint" parent="${name}_0_axel" invert="true">
+			<origin rpy="0 0 0" xyz="0 0 0" />
+		</xacro:mount_v0>
+		<xacro:drs_x01 name="${name}_1" parent="${name}_0_joint" mountBottom="false" mountBack="false" mountLeft="false" mountRight="false"
+			mountAxel="true" minPosition="${PI}" maxPosition="${PI}" maxVelocity="1">
 			<origin xyz="0 0 0" />
 		</xacro:drs_x01>
-		<xacro:drs_x01 name="${name}_2" parent="${name}_1_axel" mountBottom="true" mountBack="false" mountAxel="false" minPosition="${PI}"
-			maxPosition="${PI}" maxVelocity="1">
+		<xacro:drs_x01 name="${name}_2" parent="${name}_1_axel" mountBottom="true" mountBack="false" mountLeft="false" mountRight="false"
+			mountAxel="false" minPosition="${PI}" maxPosition="${PI}" maxVelocity="1">
 			<origin xyz="0 0 0" />
 		</xacro:drs_x01>
-		<xacro:drs_x01 name="${name}_3" parent="${name}_2_axel" mountBottom="true" mountBack="false" mountAxel="false" minPosition="${PI}"
-			maxPosition="${PI}" maxVelocity="1">
+		<xacro:drs_x01 name="${name}_3" parent="${name}_2_axel" mountBottom="true" mountBack="false" mountLeft="false" mountRight="false"
+			mountAxel="false" minPosition="${PI}" maxPosition="${PI}" maxVelocity="1">
 			<origin xyz="0 0 0" />
 		</xacro:drs_x01>

File: src/kaspar_description/urdf/kaspar_head.xacro (robot description, xacro)
@@ -34,13 +34,13 @@
 			<insert_block name="origin" />
 		</xacro:mount_point>
-		<xacro:drs_x01 name="${name}_0" mountBottom="false" mountBack="true" mountAxel="false" parent="${name}_mount" minPosition="${PI}"
-			maxPosition="${PI}" maxVelocity="1">
+		<xacro:drs_x01 name="${name}_0" parent="${name}_mount" mountBottom="false" mountBack="true" mountLeft="false" mountRight="false"
+			mountAxel="false" minPosition="${PI}" maxPosition="${PI}" maxVelocity="1">
 			<origin xyz="0 0 0" />
 		</xacro:drs_x01>
-		<xacro:drs_x01 name="${name}_1" parent="${name}_0_axel" mountBottom="true" mountBack="false" mountAxel="false" minPosition="${PI}"
-			maxPosition="${PI}" maxVelocity="1">
-			<origin xyz="0 0 0" rpy="0 0 ${PI}" />
+		<xacro:drs_x01 name="${name}_1" parent="${name}_0_axel" mountBottom="true" mountBack="false" mountLeft="false" mountRight="false"
+			mountAxel="false" minPosition="${PI}" maxPosition="${PI}" maxVelocity="1">
+			<origin xyz="0 0 0" rpy="0 0 -${PI / 2}" />
 		</xacro:drs_x01>
-		<xacro:mount_v0 name="${name}_top" parent="${name}_1_axel">
+		<xacro:mount_v0 name="${name}_top" parent="${name}_1_axel" invert="false">
 			<origin rpy="0 0 0" xyz="0 0 0" />
 		</xacro:mount_v0>

File: src/kaspar_description/urdf/kaspar_mount.xacro (robot description, xacro)
@@ -1,4 +1,5 @@
 <?xml version="1.0"?>
 <robot xmlns:xacro="http://www.ros.org/wiki/xacro">
+	<xacro:property name="VISIBLE_MOUNTS" value="true" />
 	<xacro:macro name="mount_point" params="name parent *origin">
 		<joint name="${name}_joint" type="fixed">
@@ -13,15 +14,19 @@
 				<inertia ixx="0.001" ixy="0.0" ixz="0.0" iyy="0.001" iyz="0.0" izz="0.001" />
 			</inertial>
-			<visual>
-				<origin xyz="0 0 0" rpy="0 0 0" />
-				<geometry>
-					<cylinder length="0.001" radius="0.01" />
-				</geometry>
-				<material name="mount" />
-			</visual>
+			<xacro:if value="${VISIBLE_MOUNTS}">
+				<visual>
+					<origin xyz="0 0 0" rpy="0 0 0" />
+					<geometry>
+						<cylinder length="0.001" radius="0.01" />
+					</geometry>
+					<material name="mount" />
+				</visual>
+			</xacro:if>
 		</link>
-		<gazebo reference="${name}_link">
-			<material>Gazebo/Black</material>
-		</gazebo>
+		<xacro:if value="${VISIBLE_MOUNTS}">
+			<gazebo reference="${name}_link">
+				<material>Gazebo/Black</material>
+			</gazebo>
+		</xacro:if>
 	</xacro:macro>
 </robot>

File: src/kaspar_description/urdf/kaspar_torso.xacro (robot description, xacro)
@@ -37,8 +37,8 @@
 		</xacro:mount_point>
 		<xacro:mount_point name="${name}_arm_l" parent="${name}">
-			<origin rpy="-${PI / 2} 0 0" xyz="0 0.08 0.12" />
+			<origin rpy="-${PI / 2} -${PI / 2} 0" xyz="0 0.08 0.12" />
 		</xacro:mount_point>
 		<xacro:mount_point name="${name}_arm_r" parent="${name}">
-			<origin rpy="${PI / 2} 0 0" xyz="0 -0.08 0.12" />
+			<origin rpy="${PI / 2} ${PI / 2} 0" xyz="0 -0.08 0.12" />
 		</xacro:mount_point>
 		<!-- Gazebo Config -->
