Commit message: First pass kaspar_control module, linking error in cmakefiles

File: src/kaspar_description/urdf/kaspar_arm.xacro (robot description, xacro)
@@ -40,24 +40,28 @@
 			<insert_block name="origin" />
 		</xacro:mount_point>
-		<xacro:drs_x01 name="${name}_0" parent="${name}_mount" mountBottom="false" mountBack="true" mountLeft="false" mountRight="false"
-			mountAxel="false" minPosition="${PI}" maxPosition="${PI}" maxVelocity="1">
+		<xacro:drs_x01 name="${name}_shoulder_roll_upper" parent="${name}_mount" mountBottom="false" mountBack="true" mountLeft="false"
+			mountRight="false" mountAxel="false" minPosition="${PI}" maxPosition="${PI}" maxVelocity="1">
 			<origin xyz="0 0 0" />
 		</xacro:drs_x01>
-		<xacro:mount_v0 name="${name}_0_joint" parent="${name}_0_axel" invert="true">
+		<xacro:mount_v0 name="${name}_shoulder_roll_pitch" parent="${name}_shoulder_roll_upper_axel" invert="true">
 			<origin rpy="0 0 0" xyz="0 0 0" />
 		</xacro:mount_v0>
-		<xacro:drs_x01 name="${name}_1" parent="${name}_0_joint" mountBottom="false" mountBack="false" mountLeft="false" mountRight="false"
-			mountAxel="true" minPosition="${PI}" maxPosition="${PI}" maxVelocity="1">
+		<xacro:drs_x01 name="${name}_shoulder_pitch" parent="${name}_shoulder_roll_pitch" mountBottom="true" mountBack="false"
+			mountLeft="false" mountRight="false" mountAxel="false" minPosition="${PI}" maxPosition="${PI}" maxVelocity="1">
 			<origin xyz="0 0 0" />
 		</xacro:drs_x01>
-		<xacro:drs_x01 name="${name}_2" parent="${name}_1_axel" mountBottom="true" mountBack="false" mountLeft="false" mountRight="false"
-			mountAxel="false" minPosition="${PI}" maxPosition="${PI}" maxVelocity="1">
+		<xacro:drs_x01 name="${name}_shoulder_roll_lower" parent="${name}_shoulder_pitch_axel" mountBottom="false" mountBack="false"
+			mountLeft="false" mountRight="false" mountAxel="true" minPosition="${PI}" maxPosition="${PI}" maxVelocity="1">
 			<origin xyz="0 0 0" />
 		</xacro:drs_x01>
-		<xacro:drs_x01 name="${name}_3" parent="${name}_2_axel" mountBottom="true" mountBack="false" mountLeft="false" mountRight="false"
-			mountAxel="false" minPosition="${PI}" maxPosition="${PI}" maxVelocity="1">
+		<xacro:drs_x01 name="${name}_elbow" parent="${name}_shoulder_roll_lower_axel" mountBottom="true" mountBack="false" mountLeft="false"
+			mountRight="false" mountAxel="false" minPosition="${PI}" maxPosition="${PI}" maxVelocity="1">
 			<origin xyz="0 0 0" />
 		</xacro:drs_x01>
-		<xacro:mount_point name="${name}_hand" parent="${name}_3_axel">
+		<xacro:drs_x01 name="${name}_wrist_roll" parent="${name}_elbow_axel" mountBottom="true" mountBack="false" mountLeft="false"
+			mountRight="false" mountAxel="false" minPosition="${PI}" maxPosition="${PI}" maxVelocity="1">
+			<origin xyz="0 0 0" />
+		</xacro:drs_x01>
+		<xacro:mount_point name="${name}_hand" parent="${name}_wrist_axel">
 			<origin rpy="0 0 0" xyz="0 0 0" />
 		</xacro:mount_point>

File: src/kaspar_description/urdf/kaspar_head.xacro (robot description, xacro)
@@ -34,13 +34,17 @@
 			<insert_block name="origin" />
 		</xacro:mount_point>
-		<xacro:drs_x01 name="${name}_0" parent="${name}_mount" mountBottom="false" mountBack="true" mountLeft="false" mountRight="false"
+		<xacro:drs_x01 name="${name}_yaw" parent="${name}_mount" mountBottom="false" mountBack="true" mountLeft="false" mountRight="false"
 			mountAxel="false" minPosition="${PI}" maxPosition="${PI}" maxVelocity="1">
 			<origin xyz="0 0 0" />
 		</xacro:drs_x01>
-		<xacro:drs_x01 name="${name}_1" parent="${name}_0_axel" mountBottom="true" mountBack="false" mountLeft="false" mountRight="false"
+		<xacro:drs_x01 name="${name}_pitch" parent="${name}_yaw_axel" mountBottom="true" mountBack="false" mountLeft="false" mountRight="false"
 			mountAxel="false" minPosition="${PI}" maxPosition="${PI}" maxVelocity="1">
 			<origin xyz="0 0 0" rpy="0 0 -${PI / 2}" />
 		</xacro:drs_x01>
-		<xacro:mount_v0 name="${name}_top" parent="${name}_1_axel" invert="false">
+		<xacro:drs_x01 name="${name}_roll" parent="${name}_pitch_axel" mountBottom="true" mountBack="false" mountLeft="false" mountRight="false"
+			mountAxel="false" minPosition="${PI}" maxPosition="${PI}" maxVelocity="1">
+			<origin xyz="0 0 0" rpy="0 0 -${PI / 2}" />
+		</xacro:drs_x01>
+		<xacro:mount_v0 name="${name}_top" parent="${name}_roll_axel" invert="false">
 			<origin rpy="0 0 0" xyz="0 0 0" />
 		</xacro:mount_v0>

File: src/kaspar_description/urdf/kaspar_torso.xacro (robot description, xacro)
@@ -5,5 +5,5 @@
 			<insert_block name="origin" />
 		</xacro:mount_point>
-		<joint name="${name}_joint" type="revolute">
+		<joint name="${name}_yaw_joint" type="revolute">
 			<origin xyz="0 0 0" rpy="0 0 0" />
 			<parent link="${name}_mount_link" />
@@ -43,10 +43,10 @@
 		</xacro:mount_point>
 		<!-- Gazebo Config -->
-		<transmission name="${name}_trans">
+		<transmission name="${name}_yaw_trans">
 			<type>transmission_interface/SimpleTransmission</type>
-			<joint name="${name}_joint">
+			<joint name="${name}_yaw_joint">
 				<hardwareInterface>EffortJointInterface</hardwareInterface>
 			</joint>
-			<actuator name="${name}_motor">
+			<actuator name="${name}_yaw_motor">
 				<hardwareInterface>EffortJointInterface</hardwareInterface>
 				<mechanicalReduction>1</mechanicalReduction>
